File: project-nrf-princess-dress.kicad_pcb (KiCad board)
At the start: 2 copper layers, 58 x 65 mm, 29 parts, among them J1 Conn_01x02_Female, J2 Conn_01x04_Female, J3 Conn_01x12_Female, J4 Conn_01x04_Female, J5 Conn_01x12_Female, J6 Conn_01x01_Female, J7 Conn_01x04_Female, J8 SM04B-SRSS-TB(LF)(SN), J9 Conn_01x01_Female, Q1 SI2301CDS-T1-E3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

Commit message: Save PCB in kicad 6
Other:
- net class Default removed

Commit message: Add v1.0.0 tag to silkscreen
Other:
- board text added: "Julie Gervais François Gervais 1 jan 2023 v1.0.0"
- board text removed: "Julie Gervais François Gervais 5 dec 2022 v"
Changed lines of the file:
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@@
   (gr_arc (start 99.12 24.79) (mid 101.948427 25.961573) (end 103.12 28.79) (layer "Edge.Cuts") (width 0.05))
   (gr_arc (start 49.12 89.79) (mid 46.291573 88.618427) (end 45.12 85.79) (layer "Edge.Cuts") (width 0.05))
-  (gr_text "Julie Gervais\nFrançois Gervais\n5 dec 2022\nv" (at 61.12 79.29) (layer "B.SilkS")
+  (gr_text "Julie Gervais\nFrançois Gervais\n1 jan 2023\nv1.0.0" (at 61.12 79.29) (layer "B.SilkS")
     (effects (font (size 1 1) (thickness 0.15)) (justify left mirror))
   )
